Commit message: feat: aruco planes all around the arm with proper texture

File: src/robot_description/urdf/aruco.urdf.xacro (robot description, xacro)
@@ -1,32 +1,74 @@
 <?xml version="1.0"?>
 <robot xmlns:xacro="http://www.ros.org/wiki/xacro">
-<link name="aruco_plane">
-    <visual>
-      <origin xyz="0 0 0" rpy="0 0 0"/>
-      <geometry>
-        <box size="0.1 0.1 0.001"/> <!-- 10cm x 10cm square with minimal depth (1mm) -->
-      </geometry>
-    </visual>
-    <collision>
-      <origin xyz="0 0 0" rpy="0 0 0"/>
-      <geometry>
-        <box size="0.1 0.1 0.001"/> <!-- Same as visual for collision -->
-      </geometry>
-    </collision>
-    <inertial>
-      <mass value="0.001"/> <!-- A very small mass as it's just a thin plane -->
-      <origin xyz="0 0 0" rpy="0 0 0"/>
-      <inertia ixx="0.0001" ixy="0.0" ixz="0.0"
-              iyy="0.0001" iyz="0.0" izz="0.0001"/>
-    </inertial>
-  </link>
-  <!-- Fixed joint between R5A_link5 and the plane -->
-  <joint name="aruco_plane_joint" type="fixed">
-    <parent link="R5A_link5"/> <!-- Attach to R5A_link5 -->
-    <child link="aruco_plane"/> <!-- The new plane -->
-    <origin xyz="0 0 0.2" rpy="1.57 0 0"/> <!-- Move the plane to (0, 0, 0.2) relative to R5A_link5 -->
-  </joint>
-  <gazebo reference="aruco_plane">
-    <material>Aruco0_Plane_Material</material>
-  </gazebo>
+  <!-- Xacro Macro to Define an ArUco Plane -->
+  <xacro:macro name="aruco_plane" params="plane_number parent_link position rotation">
+    <!-- Define the plane link -->
+    <link name="aruco_plane_${plane_number}">
+      <visual>
+        <origin xyz="0 0 0" rpy="0 0 0"/>
+        <geometry>
+          <box size="0.05 0.05 0.001"/> <!-- 10cm x 10cm square with minimal depth -->
+        </geometry>
+      </visual>
+      <collision>
+        <origin xyz="0 0 0" rpy="0 0 0"/>
+        <geometry>
+          <box size="0.05 0.05 0.001"/>
+        </geometry>
+      </collision>
+      <inertial>
+        <mass value="0.000001"/>
+        <origin xyz="0 0 0" rpy="0 0 0"/>
+        <inertia ixx="0.0001" ixy="0.0" ixz="0.0"
+                 iyy="0.0001" iyz="0.0" izz="0.0001"/>
+      </inertial>
+    </link>
+    <!-- Define the fixed joint attaching the plane to the parent link -->
+    <joint name="aruco_plane_joint_${plane_number}" type="fixed">
+      <parent link="${parent_link}"/>
+      <child link="aruco_plane_${plane_number}"/>
+      <origin xyz="${position}" rpy="${rotation}"/>
+    </joint>
+    <!-- Assign custom material to the plane -->
+    <gazebo reference="aruco_plane_${plane_number}">
+      <material>id${plane_number}_Plane_Material</material>
+    </gazebo>
+  </xacro:macro>
+  <!-- Instantiate the ArUco planes -->
+  <!-- For R5A_link1 -->
+  <!-- Plane 0: Front -->
+  <xacro:aruco_plane plane_number="0" parent_link="R5A_link1" position="0 0 0.1" rotation="0 0 0"/>
+  <!-- Plane 1: Back -->
+  <xacro:aruco_plane plane_number="1" parent_link="R5A_link1" position="0 0 -0.1" rotation="0 0 0"/>
+  <!-- Plane 2: Left -->
+  <xacro:aruco_plane plane_number="2" parent_link="R5A_link1" position="0.1 0 0" rotation="0 1.5708 0"/>
+  <!-- Plane 3: Right -->
+  <xacro:aruco_plane plane_number="3" parent_link="R5A_link1" position="-0.1 0 0" rotation="0 -1.5708 0"/>
+  <!-- For R5A_link2 -->
+  <!-- Plane 4: Front -->
+  <xacro:aruco_plane plane_number="4" parent_link="R5A_link2" position="0 0 0.1" rotation="0 0 0"/>
+  <!-- Plane 5: Back -->
+  <xacro:aruco_plane plane_number="5" parent_link="R5A_link2" position="0 0 -0.1" rotation="0 0 0"/>
+  <!-- Plane 6: Left -->
+  <xacro:aruco_plane plane_number="6" parent_link="R5A_link2" position="0.1 0 0" rotation="0 1.5708 0"/>
+  <!-- Plane 7: Right -->
+  <xacro:aruco_plane plane_number="7" parent_link="R5A_link2" position="-0.1 0 0" rotation="0 -1.5708 0"/>
+  <!-- For R5A_link3 -->
+  <!-- Plane 8: Front -->
+  <xacro:aruco_plane plane_number="8" parent_link="R5A_link3" position="0 0 0.05" rotation="0 0 0"/>
+  <!-- Plane 9: Back -->
+  <xacro:aruco_plane plane_number="9" parent_link="R5A_link3" position="0 0 -0.05" rotation="0 0 0"/>
+  <!-- Plane 10: Left -->
+  <xacro:aruco_plane plane_number="10" parent_link="R5A_link3" position="0.1 0 0" rotation="0 1.5708 0"/>
+  <!-- Plane 11: Right -->
+  <xacro:aruco_plane plane_number="11" parent_link="R5A_link3" position="-0.1 0 0" rotation="0 -1.5708 0"/>
+  <!-- For R5A_link4 -->
+  <!-- Plane 12: Front -->
+  <xacro:aruco_plane plane_number="12" parent_link="R5A_link4" position="0 0 0.05" rotation="0 0 0"/>
+  <!-- Plane 13: Back -->
+  <xacro:aruco_plane plane_number="13" parent_link="R5A_link4" position="0 0 -0.05" rotation="0 0 0"/>
+  <!-- Plane 14: Left -->
+  <xacro:aruco_plane plane_number="14" parent_link="R5A_link4" position="0.05 0 0" rotation="0 1.5708 0"/>
+  <!-- Plane 15: Right -->
+  <xacro:aruco_plane plane_number="15" parent_link="R5A_link4" position="-0.05 0 0" rotation="0 -1.5708 0"/>
 </robot>

Commit message: feat: implemented close-to-arm aruco planes and the right camera position

File: src/robot_description/urdf/aruco.urdf.xacro (robot description, xacro)
@@ -33,4 +33,5 @@
     <gazebo reference="aruco_plane_${plane_number}">
       <material>id${plane_number}_Plane_Material</material>
+      <disable_collision>true</disable_collision>
     </gazebo>
   </xacro:macro>
@@ -38,20 +39,20 @@
   <!-- For R5A_link1 -->
   <!-- Plane 0: Front -->
-  <xacro:aruco_plane plane_number="0" parent_link="R5A_link1" position="0 0 0.1" rotation="0 0 0"/>
+  <xacro:aruco_plane plane_number="0" parent_link="R5A_link1" position="0 0 0.08" rotation="0 0 0"/>
   <!-- Plane 1: Back -->
-  <xacro:aruco_plane plane_number="1" parent_link="R5A_link1" position="0 0 -0.1" rotation="0 0 0"/>
+  <xacro:aruco_plane plane_number="1" parent_link="R5A_link1" position="0 0 -0.08" rotation="0 0 0"/>
   <!-- Plane 2: Left -->
-  <xacro:aruco_plane plane_number="2" parent_link="R5A_link1" position="0.1 0 0" rotation="0 1.5708 0"/>
+  <xacro:aruco_plane plane_number="2" parent_link="R5A_link1" position="0.08 0 0" rotation="0 1.5708 0"/>
   <!-- Plane 3: Right -->
-  <xacro:aruco_plane plane_number="3" parent_link="R5A_link1" position="-0.1 0 0" rotation="0 -1.5708 0"/>
+  <xacro:aruco_plane plane_number="3" parent_link="R5A_link1" position="-0.08 0 0" rotation="0 -1.5708 0"/>
   <!-- For R5A_link2 -->
   <!-- Plane 4: Front -->
-  <xacro:aruco_plane plane_number="4" parent_link="R5A_link2" position="0 0 0.1" rotation="0 0 0"/>
+  <xacro:aruco_plane plane_number="4" parent_link="R5A_link2" position="0 0 0.06" rotation="0 0 0"/>
   <!-- Plane 5: Back -->
-  <xacro:aruco_plane plane_number="5" parent_link="R5A_link2" position="0 0 -0.1" rotation="0 0 0"/>
+  <xacro:aruco_plane plane_number="5" parent_link="R5A_link2" position="0 0 -0.06" rotation="0 0 0"/>
   <!-- Plane 6: Left -->
-  <xacro:aruco_plane plane_number="6" parent_link="R5A_link2" position="0.1 0 0" rotation="0 1.5708 0"/>
+  <xacro:aruco_plane plane_number="6" parent_link="R5A_link2" position="0.08 0 0" rotation="0 1.5708 0"/>
   <!-- Plane 7: Right -->
-  <xacro:aruco_plane plane_number="7" parent_link="R5A_link2" position="-0.1 0 0" rotation="0 -1.5708 0"/>
+  <xacro:aruco_plane plane_number="7" parent_link="R5A_link2" position="-0.08 0 0" rotation="0 -1.5708 0"/>
   <!-- For R5A_link3 -->
   <!-- Plane 8: Front -->
@@ -60,15 +61,15 @@
   <xacro:aruco_plane plane_number="9" parent_link="R5A_link3" position="0 0 -0.05" rotation="0 0 0"/>
   <!-- Plane 10: Left -->
-  <xacro:aruco_plane plane_number="10" parent_link="R5A_link3" position="0.1 0 0" rotation="0 1.5708 0"/>
+  <xacro:aruco_plane plane_number="10" parent_link="R5A_link3" position="0.07 0 0" rotation="0 1.5708 0"/>
   <!-- Plane 11: Right -->
-  <xacro:aruco_plane plane_number="11" parent_link="R5A_link3" position="-0.1 0 0" rotation="0 -1.5708 0"/>
+  <xacro:aruco_plane plane_number="11" parent_link="R5A_link3" position="-0.07 0 0" rotation="0 -1.5708 0"/>
   <!-- For R5A_link4 -->
   <!-- Plane 12: Front -->
-  <xacro:aruco_plane plane_number="12" parent_link="R5A_link4" position="0 0 0.05" rotation="0 0 0"/>
+  <xacro:aruco_plane plane_number="12" parent_link="R5A_link4" position="0 0.04 0.04" rotation="0 0 0"/>
   <!-- Plane 13: Back -->
-  <xacro:aruco_plane plane_number="13" parent_link="R5A_link4" position="0 0 -0.05" rotation="0 0 0"/>
+  <xacro:aruco_plane plane_number="13" parent_link="R5A_link4" position="0 0.04 -0.04" rotation="0 0 0"/>
   <!-- Plane 14: Left -->
-  <xacro:aruco_plane plane_number="14" parent_link="R5A_link4" position="0.05 0 0" rotation="0 1.5708 0"/>
+  <xacro:aruco_plane plane_number="14" parent_link="R5A_link4" position="0.042 0.04 0" rotation="0 1.5708 0"/>
   <!-- Plane 15: Right -->
-  <xacro:aruco_plane plane_number="15" parent_link="R5A_link4" position="-0.05 0 0" rotation="0 -1.5708 0"/>
+  <xacro:aruco_plane plane_number="15" parent_link="R5A_link4" position="-0.042 0.04 0" rotation="0 -1.5708 0"/>
 </robot>

File: src/robot_description/urdf/r5a_v_ros.urdf.xacro (robot description, xacro)
@@ -339,17 +339,17 @@
   <xacro:include filename="aruco.urdf.xacro" />
   <gazebo reference="base_link">
-    <material>Gazebo/White</material>
+    <material>Gazebo/Yellow</material>
   </gazebo>
   <gazebo reference="R5A_link1">
-    <material>Gazebo/White</material>
+    <material>Gazebo/Yellow</material>
   </gazebo>
   <gazebo reference="R5A_link2">
-    <material>Gazebo/White</material>
+    <material>Gazebo/Yellow</material>
   </gazebo>
   <gazebo reference="R5A_link3">
-    <material>Gazebo/White</material>
+    <material>Gazebo/Yellow</material>
   </gazebo>
   <gazebo reference="R5A_link4">
-    <material>Gazebo/White</material>
+    <material>Gazebo/Yellow</material>
   </gazebo>
   <gazebo reference="R5A_link5">
@@ -433,5 +433,5 @@
   </link>
   <joint name="camera_joint" type="fixed">
-    <origin xyz="0.5 0.5 1" rpy="1.57 1.57 0"/>
+    <origin xyz="0.6 0 0.3" rpy="0 0 3.14159"/>
       <parent link="base_link"/> <child link="camera_link"/>
   </joint>
