Commit message: feat: add camera to urdf

File: src/robot_description/urdf/r5a_v_ros.urdf.xacro (robot description, xacro)
@@ -416,3 +416,61 @@
     </plugin>
   </gazebo>
+  <!--Camera-->
+  <link name="camera_link">
+    <visual>
+      <geometry>
+        <box size="0.2 0.2 0.2"/>
+      </geometry>
+      <material name="blue"/>
+    </visual>
+    <collision>
+      <geometry>
+        <box size="0.2 0.2 0.2"/>
+      </geometry>
+    </collision>
+  </link>
+  <joint name="camera_joint" type="fixed">
+    <origin xyz="1 1 1" rpy="1.57 1.57 0"/>
+      <parent link="base_link"/> <child link="camera_link"/>
+  </joint>
+  <!--Gazebo Camera Plugin-->
+  <gazebo reference="camera_link">
+    <sensor type="camera" name="camera1">
+      <update_rate>30.0</update_rate>
+      <camera name="head">
+        <horizontal_fov>1.3962634</horizontal_fov>
+        <image>
+          <width>800</width>
+          <height>800</height>
+          <format>R8G8B8</format>
+        </image>
+        <clip>
+          <near>0.02</near>
+          <far>300</far>
+        </clip>
+        <noise>
+          <type>gaussian</type>
+          <!-- Noise is sampled independently per pixel on each frame.
+               That pixel's noise value is added to each of its color
+               channels, which at that point lie in the range [0,1]. -->
+          <mean>0.0</mean>
+          <stddev>0.007</stddev>
+        </noise>
+      </camera>
+      <plugin name="camera_controller" filename="libgazebo_ros_camera.so">
+        <alwaysOn>true</alwaysOn>
+        <updateRate>0.0</updateRate>
+        <cameraName>mybot/camera1</cameraName>
+        <imageTopicName>image_raw</imageTopicName>
+        <cameraInfoTopicName>camera_info</cameraInfoTopicName>
+        <frameName>camera_link</frameName>
+        <hackBaseline>0.07</hackBaseline>
+        <distortionK1>0.0</distortionK1>
+        <distortionK2>0.0</distortionK2>
+        <distortionK3>0.0</distortionK3>
+        <distortionT1>0.0</distortionT1>
+        <distortionT2>0.0</distortionT2>
+      </plugin>
+    </sensor>
+  </gazebo>
 </robot>

Commit message: style: moved the camera link in order for it to be closer to the arm

File: src/robot_description/urdf/r5a_v_ros.urdf.xacro (robot description, xacro)
@@ -422,5 +422,4 @@
         <box size="0.2 0.2 0.2"/>
       </geometry>
-      <material name="blue"/>
     </visual>
     <collision>
@@ -431,5 +430,5 @@
   </link>
   <joint name="camera_joint" type="fixed">
-    <origin xyz="1 1 1" rpy="1.57 1.57 0"/>
+    <origin xyz="0.5 0.5 1" rpy="1.57 1.57 0"/>
       <parent link="base_link"/> <child link="camera_link"/>
   </joint>

Commit message: fix: change camera model from box to 3D Cam mesh

File: src/robot_description/urdf/r5a_v_ros.urdf.xacro (robot description, xacro)
@@ -416,17 +416,22 @@
     </plugin>
   </gazebo>
-  <!--Camera-->
-  <link name="camera_link">
-    <visual>
-      <geometry>
-        <box size="0.2 0.2 0.2"/>
-      </geometry>
-    </visual>
-    <collision>
-      <geometry>
-        <box size="0.2 0.2 0.2"/>
-      </geometry>
-    </collision>
-  </link>
+<!-- Camera -->
+<link name="camera_link">
+  <visual>
+    <geometry>
+      <mesh filename="file://$(find robot_description)/meshes/3dCamera.DAE"/>
+    </geometry>
+    <origin rpy="0 1.5708 0"/> <!-- Rotate 90 degrees around the Y-axis (1.5708 radians = 90 degrees) -->
+  </visual>
+  <collision>
+    <geometry>
+      <mesh filename="file://$(find robot_description)/meshes/3dCamera.DAE"/>
+    </geometry>
+    <origin rpy="0 1.5708 0"/>
+  </collision>
+</link>
+<gazebo reference="camera_link">
+  <material>Gazebo/Black</material>
+</gazebo>
   <joint name="camera_joint" type="fixed">
     <origin xyz="0.5 0.5 1" rpy="1.57 1.57 0"/>

Commit message: test

File: src/robot_description/urdf/r5a_v_ros.urdf.xacro (robot description, xacro)
@@ -337,4 +337,352 @@
       velocity="1" />
   </joint>
+  <link
+    name="R5A_GripperLeft_Link1">
+    <inertial>
+      <origin
+        xyz="-0.00659452357788465 -0.000394229793384326 2.33412007907905E-06"
+        rpy="0 0 0" />
+      <mass
+        value="0.00487858122952031" />
+      <inertia
+        ixx="2.28094324920984E-07"
+        ixy="1.6939216964308E-08"
+        ixz="-1.00081436396378E-10"
+        iyy="9.51062234425376E-07"
+        iyz="1.21242073786144E-09"
+        izz="1.15060635431211E-06" />
+    </inertial>
+    <visual>
+      <origin
+        xyz="0 0 0"
+        rpy="0 0 0" />
+      <geometry>
+        <mesh
+          filename="file://$(find robot_description)/meshes/R5A_GripperLeft_Link1.STL" />
+      </geometry>
+      <material
+        name="">
+        <color
+          rgba="1 1 1 1" />
+      </material>
+    </visual>
+    <collision>
+      <origin
+        xyz="0 0 0"
+        rpy="0 0 0" />
+      <geometry>
+        <mesh
+          filename="file://$(find robot_description)/meshes/R5A_GripperLeft_Link1.STL" />
+      </geometry>
+    </collision>
+  </link>
+  <joint
+    name="ServoGearB"
+    type="revolute">
+    <origin
+      xyz="0.014 -0.00039429 0.064999"
+      rpy="1.5708 0 3.1416" />
+    <parent
+      link="R5A_link5" />
+    <child
+      link="R5A_GripperLeft_Link1" />
+    <axis
+      xyz="0 -0.006066 -0.99998" />
+      <limit
+        lower="-1.5"
+        upper="1.5"
+        effort="5"
+        velocity="1" />
+  </joint>
+  <link
+    name="R5A_GripperLeft_Link2">
+    <inertial>
+      <origin
+        xyz="0.0121769148397689 0.0264987914633754 -0.000158443058812987"
+        rpy="0 0 0" />
+      <mass
+        value="0.0102851193663261" />
+      <inertia
+        ixx="3.24436687710476E-06"
+        ixy="-1.5451128797972E-06"
+        ixz="9.58011795509406E-09"
+        iyy="1.30527398272079E-06"
+        iyz="1.62739383329679E-08"
+        izz="3.9267289910886E-06" />
+    </inertial>
+    <visual>
+      <origin
+        xyz="0 0 0"
+        rpy="0 0 0" />
+      <geometry>
+        <mesh
+          filename="file://$(find robot_description)/meshes/R5A_GripperLeft_Link2.STL" />
+      </geometry>
+      <material
+        name="">
+        <color
+          rgba="0.792156862745098 0.819607843137255 0.933333333333333 1" />
+      </material>
+    </visual>
+    <collision>
+      <origin
+        xyz="0 0 0"
+        rpy="0 0 0" />
+      <geometry>
+        <mesh
+          filename="file://$(find robot_description)/meshes/R5A_GripperLeft_Link2.STL" />
+      </geometry>
+    </collision>
+  </link>
+  <joint
+    name="LeftGripper"
+    type="revolute">
+    <origin
+      xyz="-0.04 0 0"
+      rpy="0 0 0" />
+    <parent
+      link="R5A_GripperLeft_Link1" />
+    <child
+      link="R5A_GripperLeft_Link2" />
+    <axis
+      xyz="0 -0.006066 -0.99998" />
+      <limit
+        lower="-1.5"
+        upper="1.5"
+        effort="5"
+        velocity="1" />
+  </joint>
+  <link
+    name="R5A_GripperRight_Link1">
+    <inertial>
+      <origin
+        xyz="0.00645173751342476 -0.000420742089629278 2.55112204819463E-06"
+        rpy="0 0 0" />
+      <mass
+        value="0.00500321973091749" />
+      <inertia
+        ixx="2.29355330577419E-07"
+        ixy="-1.79692415236578E-08"
+        ixz="1.09050530561434E-10"
+        iyy="9.57608070635847E-07"
+        iyz="1.21374586203517E-09"
+        izz="1.15767989130765E-06" />
+    </inertial>
+    <visual>
+      <origin
+        xyz="0 0 0"
+        rpy="0 0 0" />
+      <geometry>
+        <mesh
+          filename="file://$(find robot_description)/meshes/R5A_GripperRight_Link1.STL" />
+      </geometry>
+      <material
+        name="">
+        <color
+          rgba="1 1 1 1" />
+      </material>
+    </visual>
+    <collision>
+      <origin
+        xyz="0 0 0"
+        rpy="0 0 0" />
+      <geometry>
+        <mesh
+          filename="file://$(find robot_description)/meshes/R5A_GripperRight_Link1.STL" />
+      </geometry>
+    </collision>
+  </link>
+  <joint
+    name="IdolGearB"
+    type="revolute">
+    <origin
+      xyz="-0.014 -0.00039429 0.064999"
+      rpy="1.5708 0 3.1416" />
+    <parent
+      link="R5A_link5" />
+    <child
+      link="R5A_GripperRight_Link1" />
+    <axis
+      xyz="0 -0.006066 -0.99998" />
+      <limit
+        lower="-1.5"
+        upper="1.5"
+        effort="5"
+        velocity="1" />
+  </joint>
+  <link
+    name="R5A_GripperRight_Link12">
+    <inertial>
+      <origin
+        xyz="-0.0121769121022422 0.0264987629996978 -0.000158239935640828"
+        rpy="0 0 0" />
+      <mass
+        value="0.0102851432058251" />
+      <inertia
+        ixx="3.24437190589206E-06"
+        ixy="1.54511360510839E-06"
+        ixz="-9.56821825774594E-09"
+        iyy="1.3052751101257E-06"
+        iyz="1.63061443850097E-08"
+        izz="3.92673308798734E-06" />
+    </inertial>
+    <visual>
+      <origin
+        xyz="0 0 0"
+        rpy="0 0 0" />
+      <geometry>
+        <mesh
+          filename="file://$(find robot_description)/meshes/R5A_GripperRight_Link12.STL" />
+      </geometry>
+      <material
+        name="">
+        <color
+          rgba="0.792156862745098 0.819607843137255 0.933333333333333 1" />
+      </material>
+    </visual>
+    <collision>
+      <origin
+        xyz="0 0 0"
+        rpy="0 0 0" />
+      <geometry>
+        <mesh
+          filename="file://$(find robot_description)/meshes/R5A_GripperRight_Link12.STL" />
+      </geometry>
+    </collision>
+  </link>
+  <joint
+    name="RightGripper"
+    type="revolute">
+    <origin
+      xyz="0.04 -8.7393E-05 0"
+      rpy="0 0 0" />
+    <parent
+      link="R5A_GripperRight_Link1" />
+    <child
+      link="R5A_GripperRight_Link12" />
+    <axis
+      xyz="0 -0.006066 -0.99998" />
+      <limit
+        lower="-1.5"
+        upper="1.5"
+        effort="5"
+        velocity="1" />
+  </joint>
+  <link
+    name="R5A_GripperLeft_Link3">
+    <inertial>
+      <origin
+        xyz="-0.0199999997525655 3.145952191419E-06 -1.90838667814405E-08"
+        rpy="0 0 0" />
+      <mass
+        value="0.00167027391699935" />
+      <inertia
+        ixx="1.05068364831453E-08"
+        ixy="4.70838754646646E-11"
+        ixz="-2.8561858514888E-13"
+        iyy="3.09836744743031E-07"
+        iyz="5.57882383977291E-12"
+        izz="3.1075637533632E-07" />
+    </inertial>
+    <visual>
+      <origin
+        xyz="0 0 0"
+        rpy="0 0 0" />
+      <geometry>
+        <mesh
+          filename="file://$(find robot_description)/meshes/R5A_GripperLeft_Link3.STL" />
+      </geometry>
+      <material
+        name="">
+        <color
+          rgba="1 1 1 1" />
+      </material>
+    </visual>
+    <collision>
+      <origin
+        xyz="0 0 0"
+        rpy="0 0 0" />
+      <geometry>
+        <mesh
+          filename="file://$(find robot_description)/meshes/R5A_GripperLeft_Link3.STL" />
+      </geometry>
+    </collision>
+  </link>
+  <joint
+    name="LeftPivotArm"
+    type="revolute">
+    <origin
+      xyz="0.007 -0.00051561 0.084998"
+      rpy="1.5708 0 3.1416" />
+    <parent
+      link="R5A_link5" />
+    <child
+      link="R5A_GripperLeft_Link3" />
+    <axis
+      xyz="0 0.006066 0.99998" />
+      <limit
+        lower="-1.5"
+        upper="1.5"
+        effort="5"
+        velocity="1" />
+  </joint>
+  <link
+    name="R5A_GripperRight_Link3">
+    <inertial>
+      <origin
+        xyz="0.0199999522632083 -4.36966718125875E-05 2.65070677342503E-07"
+        rpy="0 0 0" />
+      <mass
+        value="0.00167027391699936" />
+      <inertia
+        ixx="1.05082579798441E-08"
+        ixy="6.53984435711306E-10"
+        ixz="-3.96716935939432E-12"
+        iyy="3.09835323298639E-07"
+        iyz="5.5874465381491E-12"
+        izz="3.10756375284014E-07" />
+    </inertial>
+    <visual>
+      <origin
+        xyz="0 0 0"
+        rpy="0 0 0" />
+      <geometry>
+        <mesh
+          filename="file://$(find robot_description)/meshes/R5A_GripperRight_Link3.STL" />
+      </geometry>
+      <material
+        name="">
+        <color
+          rgba="1 1 1 1" />
+      </material>
+    </visual>
+    <collision>
+      <origin
+        xyz="0 0 0"
+        rpy="0 0 0" />
+      <geometry>
+        <mesh
+          filename="file://$(find robot_description)/meshes/R5A_GripperRight_Link3.STL" />
+      </geometry>
+    </collision>
+  </link>
+  <joint
+    name="RigtPivotArm"
+    type="revolute">
+    <origin
+      xyz="-0.007 -0.00051561 0.084998"
+      rpy="1.5708 0 3.1416" />
+    <parent
+      link="R5A_link5" />
+    <child
+      link="R5A_GripperRight_Link3" />
+    <axis
+      xyz="0 -0.006066 -0.99998" />
+      <limit
+        lower="-1.5"
+        upper="1.5"
+        effort="5"
+        velocity="1" />
+  </joint>
   <gazebo reference="base_link">
     <material>Gazebo/White</material>
@@ -353,4 +701,22 @@
   </gazebo>
   <gazebo reference="R5A_link5">
+    <material>Gazebo/Black</material>
+  </gazebo>
+  <gazebo reference="R5A_GripperRight_Link1">
+    <material>Gazebo/Black</material>
+  </gazebo>
+  <gazebo reference="R5A_GripperRight_Link12">
+    <material>Gazebo/Black</material>
+  </gazebo>
+  <gazebo reference="R5A_GripperRight_Link3">
+    <material>Gazebo/Black</material>
+  </gazebo>
+  <gazebo reference="R5A_GripperLeft_Link1">
+    <material>Gazebo/Black</material>
+  </gazebo>
+  <gazebo reference="R5A_GripperLeft_Link2">
+    <material>Gazebo/Black</material>
+  </gazebo>
+  <gazebo reference="R5A_GripperLeft_Link3">
     <material>Gazebo/Black</material>
   </gazebo>
@@ -359,4 +725,5 @@
       <plugin>gazebo_ros2_control/GazeboSystem</plugin>
     </hardware>
+    <!-- Arm Joints -->
     <joint name="R0_Yaw">
       <command_interface name="position"/>
@@ -388,4 +755,47 @@
     </joint>
     <joint name="R4_Pitch">
+      <command_interface name="position"/>
+      <state_interface name="position">
+        <param name="initial_value">0.0</param>
+      </state_interface>
+      <state_interface name="velocity"/>
+    </joint>
+    <!-- Gripper Joints -->
+    <joint name="ServoGearB">
+      <command_interface name="position"/>
+      <state_interface name="position">
+        <param name="initial_value">0.0</param>
+      </state_interface>
+      <state_interface name="velocity"/>
+    </joint>
+    <joint name="LeftGripper">
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
Commit message: feat: add second camera

File: src/robot_description/urdf/r5a_v_ros.urdf.xacro (robot description, xacro)
@@ -416,31 +416,32 @@
     </plugin>
   </gazebo>
-<!-- Camera -->
-<link name="camera_link">
-  <visual>
-    <geometry>
-      <mesh filename="file://$(find robot_description)/meshes/3dCamera.DAE"/>
-    </geometry>
-    <origin rpy="0 1.5708 0"/> <!-- Rotate 90 degrees around the Y-axis (1.5708 radians = 90 degrees) -->
-  </visual>
-  <collision>
-    <geometry>
-      <mesh filename="file://$(find robot_description)/meshes/3dCamera.DAE"/>
-    </geometry>
-    <origin rpy="0 1.5708 0"/>
-  </collision>
-</link>
-<gazebo reference="camera_link">
-  <material>Gazebo/Black</material>
-</gazebo>
-  <joint name="camera_joint" type="fixed">
+<!-- First Camera -->
+  <link name="camera_link1">
+    <visual>
+      <geometry>
+        <mesh filename="file://$(find robot_description)/meshes/3dCamera.DAE"/>
+      </geometry>
+      <origin rpy="0 1.5708 0"/> <!-- Rotate 90 degrees around the Y-axis (1.5708 radians = 90 degrees) -->
+    </visual>
+    <collision>
+      <geometry>
+        <mesh filename="file://$(find robot_description)/meshes/3dCamera.DAE"/>
+      </geometry>
+      <origin rpy="0 1.5708 0"/>
+    </collision>
+  </link>
+  <gazebo reference="camera_link1">
+    <material>Gazebo/Black</material>
+  </gazebo>
+  <joint name="camera_joint1" type="fixed">
     <origin xyz="0.5 0.5 1" rpy="1.57 1.57 0"/>
-      <parent link="base_link"/> <child link="camera_link"/>
-  </joint>
-  <!--Gazebo Camera Plugin-->
-  <gazebo reference="camera_link">
+    <parent link="base_link"/>
+    <child link="camera_link1"/>
+  </joint>
+  <!-- Gazebo Camera Plugin for First Camera -->
+  <gazebo reference="camera_link1">
     <sensor type="camera" name="camera1">
       <update_rate>30.0</update_rate>
-      <camera name="head">
+      <camera name="head1">
         <horizontal_fov>1.3962634</horizontal_fov>
         <image>
@@ -455,12 +456,9 @@
         <noise>
           <type>gaussian</type>
-          <!-- Noise is sampled independently per pixel on each frame.
-               That pixel's noise value is added to each of its color
-               channels, which at that point lie in the range [0,1]. -->
           <mean>0.0</mean>
           <stddev>0.007</stddev>
         </noise>
       </camera>
-      <plugin name="camera_controller" filename="libgazebo_ros_camera.so">
+      <plugin name="camera_controller1" filename="libgazebo_ros_camera.so">
         <alwaysOn>true</alwaysOn>
         <updateRate>0.0</updateRate>
@@ -468,5 +466,5 @@
         <imageTopicName>image_raw</imageTopicName>
         <cameraInfoTopicName>camera_info</cameraInfoTopicName>
-        <frameName>camera_link</frameName>
+        <frameName>camera_link1</frameName>
         <hackBaseline>0.07</hackBaseline>
         <distortionK1>0.0</distortionK1>
@@ -478,3 +476,63 @@
     </sensor>
   </gazebo>
+  <!-- Second Camera -->
+  <link name="camera_link2">
+    <visual>
+      <geometry>
+        <mesh filename="file://$(find robot_description)/meshes/3dCamera.DAE"/>
+      </geometry>
+      <origin rpy="0 1.5708 0"/> <!-- Rotate 90 degrees around the Y-axis (1.5708 radians = 90 degrees) -->
+    </visual>
+    <collision>
+      <geometry>
+        <mesh filename="file://$(find robot_description)/meshes/3dCamera.DAE"/>
+      </geometry>
+      <origin rpy="0 1.5708 0"/>
+    </collision>
+  </link>
+  <gazebo reference="camera_link2">
+    <material>Gazebo/Black</material>
+  </gazebo>
+  <joint name="camera_joint2" type="fixed">
+    <origin xyz="-0.5 0.5 1" rpy="1.57 1.57 0"/> <!-- Adjust xyz to place in front of the first camera -->
+    <parent link="base_link"/>
+    <child link="camera_link2"/>
+  </joint>
+  <!-- Gazebo Camera Plugin for Second Camera -->
+  <gazebo reference="camera_link2">
+    <sensor type="camera" name="camera2">
+      <update_rate>30.0</update_rate>
+      <camera name="head2">
+        <horizontal_fov>1.3962634</horizontal_fov>
+        <image>
+          <width>800</width>
+          <height>800</height>
+          <format>R8G8B8</format>
+        </image>
+        <clip>
+          <near>0.02</near>
+          <far>300</far>
+        </clip>
+        <noise>
+          <type>gaussian</type>
+          <mean>0.0</mean>
+          <stddev>0.007</stddev>
+        </noise>
+      </camera>
+      <plugin name="camera_controller2" filename="libgazebo_ros_camera.so">
+        <alwaysOn>true</alwaysOn>
+        <updateRate>0.0</updateRate>
+        <cameraName>mybot/camera2</cameraName>
+        <imageTopicName>image_raw2</imageTopicName>
+        <cameraInfoTopicName>camera_info2</cameraInfoTopicName>
+        <frameName>camera_link2</frameName>
+        <hackBaseline>0.07</hackBaseline>
+        <distortionK1>0.0</distortionK1>
+        <distortionK2>0.0</distortionK2>
+        <distortionK3>0.0</distortionK3>
+        <distortionT1>0.0</distortionT1>
+        <distortionT2>0.0</distortionT2>
+      </plugin>
+    </sensor>
+  </gazebo>
 </robot>
