Commit message: feat: add gripper functionalities in URDF

File: src/robot_description/urdf/r5a_v_ros.urdf.xacro (robot description, xacro)
@@ -1,4 +1,5 @@
 <?xml version="1.0" encoding="utf-8"?>
 <robot name="armr5" xmlns:xacro="http://www.ros.org/wiki/xacro">
+  <xacro:include filename="aruco.urdf.xacro" />
   <link name="world"></link>
   <joint name="base_joint" type="fixed">
@@ -17,8 +18,8 @@
       <inertia
         ixx="0.00335325507409126"
-        ixy="-2.74339673314697E-05"
-        ixz="6.86594556641863E-08"
+        ixy="-2.743396733147E-05"
+        ixz="6.86594556642029E-08"
         iyy="0.00381821146815156"
-        iyz="-1.94234209654721E-06"
+        iyz="-1.9423420965472E-06"
         izz="0.00646111115889031" />
     </inertial>
@@ -51,5 +52,5 @@
     <inertial>
       <origin
-        xyz="-0.000863539879134232 0.0792884229151366 0.000217126309188392"
+        xyz="-0.000863539879134213 0.0792884229151367 0.000217126309188408"
         rpy="0 0 0" />
       <mass
@@ -57,8 +58,8 @@
       <inertia
         ixx="0.00705202984610834"
-        ixy="4.18495769538317E-07"
-        ixz="-5.35090527847856E-08"
+        ixy="4.18495769536855E-07"
+        ixz="-5.35090527857546E-08"
         iyy="0.00650257727022909"
-        iyz="-7.95450001919316E-07"
+        iyz="-7.95450001919519E-07"
         izz="0.00859235014286563" />
     </inertial>
@@ -109,15 +110,15 @@
     <inertial>
       <origin
-        xyz="0.000590340031700868 0.0792749789345379 -1.60575865215957E-05"
+        xyz="0.000590340031700784 0.0792749789345383 -1.60575865215828E-05"
         rpy="0 0 0" />
       <mass
         value="1.92247082198063" />
       <inertia
-        ixx="0.00487699383852878"
-        ixy="-3.6797699062717E-05"
-        ixz="1.05680472821036E-06"
-        iyy="0.002932746016665"
-        iyz="-4.85804534873411E-08"
-        izz="0.00503562271238705" />
+        ixx="0.00487699383852877"
+        ixy="-3.67976990627086E-05"
+        ixz="1.05680472821134E-06"
+        iyy="0.00293274601666501"
+        iyz="-4.85804534901831E-08"
+        izz="0.00503562271238706" />
     </inertial>
     <visual>
@@ -149,5 +150,5 @@
     type="revolute">
     <origin
-      xyz="-0.00310901547925539 0.1655 0"
+      xyz="-0.00310901547925538 0.1655 0"
       rpy="0 0 0" />
     <parent
@@ -156,5 +157,5 @@
       link="R5A_link2" />
     <axis
-      xyz="-1 0 0" />
+      xyz="-0.999934112328875 0 -0.011479155067573" />
     <limit
       lower="-1.5"
@@ -167,14 +168,14 @@
     <inertial>
       <origin
-        xyz="-0.000315549279166808 0.0424449594079959 0.000423163095624355"
-        rpy="0 0 0" />
-      <mass
-        value="0.749292336081854" />
+        xyz="-0.000315549279166789 0.042444959407996 0.00042316309562433"
+        rpy="0 0 0" />
+      <mass
+        value="0.749292336081855" />
       <inertia
         ixx="0.00200425601332893"
-        ixy="9.17956375018228E-06"
-        ixz="-2.55766332055333E-08"
-        iyy="0.00069735819745095"
-        iyz="-7.84063656624613E-06"
+        ixy="9.1795637501825E-06"
+        ixz="-2.55766332056785E-08"
+        iyy="0.000697358197450952"
+        iyz="-7.84063656624641E-06"
         izz="0.00196480563389349" />
     </inertial>
@@ -215,5 +216,5 @@
     <axis
       xyz="-1 0 0" />
-   <limit
+    <limit
       lower="-1.5"
       upper="1.5"
@@ -225,15 +226,15 @@
     <inertial>
       <origin
-        xyz="-0.000206047771173058 0.0454873904143689 -0.000219105733635074"
-        rpy="0 0 0" />
-      <mass
-        value="0.355077243317324" />
-      <inertia
-        ixx="0.000669805200122677"
-        ixy="-4.71996739328152E-07"
-        ixz="-1.57736445618108E-07"
-        iyy="0.000358674558440702"
-        iyz="-5.41990969302289E-08"
-        izz="0.00076811625156356" />
+        xyz="-0.000206047771187218 0.0454873904143415 -0.000219105733632293"
+        rpy="0 0 0" />
+      <mass
+        value="0.355077243317478" />
+      <inertia
+        ixx="0.000669805200123062"
+        ixy="-4.71996739637697E-07"
+        ixz="-1.57736445584604E-07"
+        iyy="0.000358674558440891"
+        iyz="-5.41990968682589E-08"
+        izz="0.000768116251564114" />
     </inertial>
     <visual>
@@ -272,5 +273,5 @@
       link="R5A_link4" />
     <axis
-      xyz="0 -1 0" />
+      xyz="0 -0.999718303067734 -0.0237342476470231" />
     <limit
       lower="-1.5"
@@ -283,15 +284,15 @@
     <inertial>
       <origin
-        xyz="-0.000304982815722917 0.000214555031841958 0.0238812711123602"
-        rpy="0 0 0" />
-      <mass
-        value="0.232244400597819" />
-      <inertia
-        ixx="0.000120322215361587"
-        ixy="-9.01049257248474E-08"
-        ixz="2.57785604684289E-07"
-        iyy="9.55044143695027E-05"
-        iyz="-7.60482494086889E-08"
-        izz="6.98522198363616E-05" />
+        xyz="-0.000347552332670687 0.000167028378251888 0.0138173380766619"
+        rpy="0 0 0" />
+      <mass
+        value="0.198451767848984" />
+      <inertia
+        ixx="0.000113354976202718"
+        ixy="-9.1633661632938E-08"
+        ixz="2.54500165125599E-07"
+        iyy="8.47211726683811E-05"
+        iyz="4.4543875805716E-08"
+        izz="6.47134110451793E-05" />
     </inertial>
     <visual>
@@ -306,4 +307,62 @@
         name="">
         <color
+          rgba="0.792156862745098 0.819607843137255 0.933333333333333 1" />
+      </material>
+    </visual>
+    <collision>
+      <origin
+        xyz="0 0 0"
+        rpy="0 0 0" />
+      <geometry>
+        <mesh
+          filename="file://$(find robot_description)/meshes/R5A_link5.STL" />
+      </geometry>
+    </collision>
+  </link>
+  <joint
+    name="R4_Pitch"
+    type="revolute">
+    <origin
+      xyz="0 0.0950000000000002 0"
+      rpy="1.5707963267949 0 3.14159265358979" />
+    <parent
+      link="R5A_link4" />
+    <child
+      link="R5A_link5" />
+    <axis
+      xyz="-0.995634790742834 0.0933346852058426 0" />
+    <limit
+      lower="-1.5"
+      upper="1.5"
+      effort="5"
+      velocity="1" />
+  </joint>
+  <link
+    name="R5A_GripperLeft_Link1">
+    <inertial>
+      <origin
+        xyz="-0.00659452357779758 -0.000394229793377554 2.33412007890428E-06"
+        rpy="0 0 0" />
+      <mass
+        value="0.00487858122952023" />
+      <inertia
+        ixx="2.28094324920978E-07"
+        ixy="1.69392169643129E-08"
+        ixz="-1.00081436396101E-10"
+        iyy="9.51062234425361E-07"
+        iyz="1.21242073786193E-09"
+        izz="1.15060635431209E-06" />
+    </inertial>
+    <visual>
+      <origin
+        xyz="0 0 0"
+        rpy="0 0 0" />
+      <geometry>
+        <mesh
+          filename="file://$(find robot_description)/meshes/R5A_GripperLeft_Link1.STL" />
+      </geometry>
+      <material
+        name="">
+        <color
           rgba="1 1 1 1" />
       </material>
@@ -315,27 +374,316 @@
       <geometry>
         <mesh
-          filename="file://$(find robot_description)/meshes/R5A_link5.STL" />
-      </geometry>
-    </collision>
-  </link>
-  <joint
-    name="R4_Pitch"
-    type="revolute">
-    <origin
-      xyz="0 0.095 0"
+          filename="file://$(find robot_description)/meshes/R5A_GripperLeft_Link1.STL" />
+      </geometry>
+    </collision>
+  </link>
+  <joint
+    name="ServoGearB"
+    type="revolute">
+    <origin
+      xyz="0.0140000000000435 -0.000394292596204153 0.0649988040916903"
+      rpy="1.5707963267949 0 3.14159265358979" />
+    <parent
+      link="R5A_link5" />
+    <child
+      link="R5A_GripperLeft_Link1" />
+    <axis
+      xyz="0 -0.006066039941515 -0.99998160141046" />
+    <limit
+      lower="-1.5"
+      upper="1.5"
+      effort="5"
+      velocity="1" />
+  </joint>
+  <link
+    name="R5A_GripperLeft_Link2">
+    <inertial>
+      <origin
+        xyz="0.0121769148397674 0.0264987914633908 -0.00015844305881356"
+        rpy="0 0 0" />
+      <mass
+        value="0.010285119366326" />
+      <inertia
+        ixx="3.24436687710476E-06"
+        ixy="-1.54511287979719E-06"
+        ixz="9.58011795509873E-09"
+        iyy="1.30527398272079E-06"
+        iyz="1.62739383329718E-08"
+        izz="3.9267289910886E-06" />
+    </inertial>
+    <visual>
+      <origin
+        xyz="0 0 0"
+        rpy="0 0 0" />
+      <geometry>
+        <mesh
+          filename="file://$(find robot_description)/meshes/R5A_GripperLeft_Link2.STL" />
+      </geometry>
+      <material
+        name="">
+        <color
+          rgba="0.792156862745098 0.819607843137255 0.933333333333333 1" />
+      </material>
+    </visual>
+    <collision>
+      <origin
+        xyz="0 0 0"
+        rpy="0 0 0" />
+      <geometry>
+        <mesh
+          filename="file://$(find robot_description)/meshes/R5A_GripperLeft_Link2.STL" />
+      </geometry>
+    </collision>
+  </link>
+  <joint
+    name="LeftGripper"
+    type="revolute">
+    <origin
+      xyz="-0.0399999995050676 0 0"
+      rpy="0 0 0" />
+    <parent
+      link="R5A_GripperLeft_Link1" />
+    <child
+      link="R5A_GripperLeft_Link2" />
+    <axis
+      xyz="0 -0.00606603994152109 -0.99998160141046" />
+    <limit
+      lower="-1.5"
+      upper="1.5"
+      effort="5"
+      velocity="1" />
+  </joint>
+  <link
+    name="R5A_GripperRight_Link1">
+    <inertial>
+      <origin
+        xyz="0.00645173751362635 -0.000420742089632498 2.55112204775943E-06"
+        rpy="0 0 0" />
+      <mass
+        value="0.0050032197309173" />
+      <inertia
+        ixx="2.29355330577406E-07"
+        ixy="-1.79692415236652E-08"
+        ixz="1.09050530560748E-10"
+        iyy="9.5760807063583E-07"
+        iyz="1.21374586203625E-09"
+        izz="1.15767989130762E-06" />
+    </inertial>
+    <visual>
+      <origin
+        xyz="0 0 0"
+        rpy="0 0 0" />
+      <geometry>
+        <mesh
+          filename="file://$(find robot_description)/meshes/R5A_GripperRight_Link1.STL" />
+      </geometry>
+      <material
+        name="">
+        <color
+          rgba="1 1 1 1" />
+      </material>
+    </visual>
+    <collision>
+      <origin
+        xyz="0 0 0"
+        rpy="0 0 0" />
+      <geometry>
+        <mesh
+          filename="file://$(find robot_description)/meshes/R5A_GripperRight_Link1.STL" />
+      </geometry>
+    </collision>
+  </link>
+  <joint
+    name="IdolGearB"
+    type="revolute">
+    <origin
+      xyz="-0.014 -0.00039429 0.064999"
       rpy="1.5708 0 3.1416" />
     <parent
-      link="R5A_link4" />
-    <child
       link="R5A_link5" />
-    <axis
-      xyz="-1 0 0" />
-    <limit
-      lower="-1.5"
-      upper="1.5"
-      effort="5"
-      velocity="1" />
-  </joint>
-  <xacro:include filename="aruco.urdf.xacro" />
+    <child
+      link="R5A_GripperRight_Link1" />
+    <axis
+      xyz="0 -0.006066 -0.99998" />
+    <limit
+      lower="-1.5"
+      upper="1.5"
+      effort="5"
+      velocity="1" />
+  </joint>
+  <link
+    name="R5A_GripperRight_Link12">
+    <inertial>
+      <origin
+        xyz="-0.0121769121022437 0.0264987629997102 -0.000158239935641401"
+        rpy="0 0 0" />
+      <mass
+        value="0.010285143205825" />
+      <inertia
+        ixx="3.24437190589205E-06"
+        ixy="1.54511360510839E-06"
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
Commit message: mod

File: src/robot_description/urdf/r5a_v_ros.urdf.xacro (robot description, xacro)
@@ -4,5 +4,5 @@
   <link name="world"></link>
   <joint name="base_joint" type="fixed">
-    <origine xyz="0 0 0" rpy="0 0 0"/>
+    <origin xyz="0 0 0" rpy="0 0 0"/>
     <parent link="world"/>
     <child link="base_link"/>
@@ -669,5 +669,5 @@
   </link>
   <joint
-    name="RigtPivotArm"
+    name="RightPivotArm"
     type="revolute">
     <origin

File: src/robot_moveit_config/config/armr5.ros2_control.xacro (robot description, xacro)
@@ -43,4 +43,46 @@
                 <state_interface name="velocity"/>
             </joint>
+            <joint name="IdolGearB">
+                <command_interface name="position"/>
+                <state_interface name="position">
+                  <param name="initial_value">${initial_positions['IdolGearB']}</param>
+                </state_interface>
+                <state_interface name="velocity"/>
+            </joint>
+            <joint name="RightGripper">
+                <command_interface name="position"/>
+                <state_interface name="position">
+                  <param name="initial_value">${initial_positions['RightGripper']}</param>
+                </state_interface>
+                <state_interface name="velocity"/>
+            </joint>
+            <joint name="LeftPivotArm">
+                <command_interface name="position"/>
+                <state_interface name="position">
+                  <param name="initial_value">${initial_positions['LeftPivotArm']}</param>
+                </state_interface>
+                <state_interface name="velocity"/>
+            </joint>
+            <joint name="RightPivotArm">
+                <command_interface name="position"/>
+                <state_interface name="position">
+                  <param name="initial_value">${initial_positions['RightPivotArm']}</param>
+                </state_interface>
+                <state_interface name="velocity"/>
+            </joint>
+            <joint name="ServoGearB">
+                <command_interface name="position"/>
+                <state_interface name="position">
+                  <param name="initial_value">${initial_positions['ServoGearB']}</param>
+                </state_interface>
+                <state_interface name="velocity"/>
+            </joint>
+            <joint name="LeftGripper">
+                <command_interface name="position"/>
+                <state_interface name="position">
+                  <param name="initial_value">${initial_positions['LeftGripper']}</param>
+                </state_interface>
+                <state_interface name="velocity"/>
+            </joint>
         </ros2_control>
     </xacro:macro>

Commit message: Gripper Mimic

File: src/robot_description/urdf/r5a_v_ros.urdf.xacro (robot description, xacro)
@@ -379,5 +379,5 @@
   </link>
   <joint
-    name="ServoGearB"
+    name="ServoGear"
     type="revolute">
     <origin
@@ -453,4 +453,5 @@
       effort="5"
       velocity="1" />
+    <mimic joint="ServoGear" multiplier="-1"/>
   </joint>
   <link
@@ -495,5 +496,5 @@
   </link>
   <joint
-    name="IdolGearB"
+    name="PassifGear"
     type="revolute">
     <origin
@@ -511,4 +512,5 @@
       effort="5"
       velocity="1" />
+    <mimic joint="ServoGear" multiplier="-1"/>
   </joint>
   <link
@@ -569,4 +571,5 @@
       effort="5"
       velocity="1" />
+    <mimic joint="ServoGear" multiplier="1"/>
   </joint>
   <link
@@ -627,4 +630,5 @@
       effort="5"
       velocity="1" />
+    <mimic joint="ServoGear" multiplier="-1"/>
   </joint>
   <link
@@ -685,4 +689,5 @@
       effort="5"
       velocity="1" />
+    <mimic joint="ServoGear" multiplier="-1"/>
   </joint>
   <gazebo reference="base_link">
@@ -703,4 +708,22 @@
   <gazebo reference="R5A_link5">
     <material>Gazebo/Black</material>
+  </gazebo>
+  <gazebo reference="R5A_GripperRight_Link1">
+    <material>Gazebo/White</material>
+  </gazebo>
+  <gazebo reference="R5A_GripperRight_Link2">
+    <material>Gazebo/Black</material>
+  </gazebo>
+  <gazebo reference="R5A_GripperRight_Link3">
+    <material>Gazebo/White</material>
+  </gazebo>
+  <gazebo reference="R5A_GripperLeft_Link1">
+    <material>Gazebo/White</material>
+  </gazebo>
+  <gazebo reference="R5A_GripperLeft_Link2">
+    <material>Gazebo/Black</material>
+  </gazebo>
+  <gazebo reference="R5A_GripperLeft_Link3">
+    <material>Gazebo/White</material>
   </gazebo>
   <ros2_control name="GazeboSystem" type="system">
@@ -738,4 +761,46 @@
     </joint>
     <joint name="R4_Pitch">
+      <command_interface name="position"/>
+      <state_interface name="position">
+        <param name="initial_value">0.0</param>
+      </state_interface>
+      <state_interface name="velocity"/>
+    </joint>
+    <joint name="ServoGear">
+      <command_interface name="position"/>
+      <state_interface name="position">
+        <param name="initial_value">0.0</param>
+      </state_interface>
+      <state_interface name="velocity"/>
+    </joint>
+    <joint name="LeftGripper">
+      <command_interface name="position"/>
+      <state_interface name="position">
+        <param name="initial_value">0.0</param>
+      </state_interface>
+      <state_interface name="velocity"/>
+    </joint>
+    <joint name="LeftPivotArm">
+      <command_interface name="position"/>
+      <state_interface name="position">
+        <param name="initial_value">0.0</param>
+      </state_interface>
+      <state_interface name="velocity"/>
+    </joint>
+    <joint name="PassifGear">
+      <command_interface name="position"/>
+      <state_interface name="position">
+        <param name="initial_value">0.0</param>
+      </state_interface>
+      <state_interface name="velocity"/>
+    </joint>
+    <joint name="RightGripper">
+      <command_interface name="position"/>
+      <state_interface name="position">
+        <param name="initial_value">0.0</param>
+      </state_interface>
+      <state_interface name="velocity"/>
+    </joint>
+    <joint name="RightPivotArm">
       <command_interface name="position"/>
       <state_interface name="position">
@@ -765,4 +830,10 @@
         <joint_name>R3_Yaw</joint_name>
         <joint_name>R4_Pitch</joint_name>
+        <joint_name>ServoGear</joint_name>
+        <joint_name>LeftGripper</joint_name>
+        <joint_name>LeftPivotArm</joint_name>
+        <joint_name>PassifGear</joint_name>
+        <joint_name>RightGripper</joint_name>
+        <joint_name>RightPivotArm</joint_name>
     </plugin>
   </gazebo>

File: src/robot_moveit_config/config/armr5.ros2_control.xacro (robot description, xacro)
@@ -43,43 +43,8 @@
                 <state_interface name="velocity"/>
             </joint>
-            <joint name="IdolGearB">
+            <joint name="ServoGear">
                 <command_interface name="position"/>
                 <state_interface name="position">
-                  <param name="initial_value">${initial_positions['IdolGearB']}</param>
-                </state_interface>
-                <state_interface name="velocity"/>
-            </joint>
-            <joint name="RightGripper">
-                <command_interface name="position"/>
-                <state_interface name="position">
-                  <param name="initial_value">${initial_positions['RightGripper']}</param>
-                </state_interface>
-                <state_interface name="velocity"/>
-            </joint>
-            <joint name="LeftPivotArm">
-                <command_interface name="position"/>
-                <state_interface name="position">
-                  <param name="initial_value">${initial_positions['LeftPivotArm']}</param>
-                </state_interface>
-                <state_interface name="velocity"/>
-            </joint>
-            <joint name="RightPivotArm">
-                <command_interface name="position"/>
-                <state_interface name="position">
-                  <param name="initial_value">${initial_positions['RightPivotArm']}</param>
-                </state_interface>
-                <state_interface name="velocity"/>
-            </joint>
-            <joint name="ServoGearB">
-                <command_interface name="position"/>
-                <state_interface name="position">
-                  <param name="initial_value">${initial_positions['ServoGearB']}</param>
-                </state_interface>
-                <state_interface name="velocity"/>
-            </joint>
-            <joint name="LeftGripper">
-                <command_interface name="position"/>
-                <state_interface name="position">
-                  <param name="initial_value">${initial_positions['LeftGripper']}</param>
+                  <param name="initial_value">${initial_positions['ServoGear']}</param>
                 </state_interface>
                 <state_interface name="velocity"/>

Commit message: Gripper controlable but no mimic only hard code

File: src/robot_description/urdf/r5a_v_ros.urdf.xacro (robot description, xacro)
@@ -453,5 +453,4 @@
       effort="5"
       velocity="1" />
-    <mimic joint="ServoGear" multiplier="-1"/>
   </joint>
   <link
@@ -512,5 +511,4 @@
       effort="5"
       velocity="1" />
-    <mimic joint="ServoGear" multiplier="-1"/>
   </joint>
   <link
@@ -571,5 +569,4 @@
       effort="5"
       velocity="1" />
-    <mimic joint="ServoGear" multiplier="1"/>
   </joint>
   <link
@@ -630,5 +627,4 @@
       effort="5"
       velocity="1" />
-    <mimic joint="ServoGear" multiplier="-1"/>
   </joint>
   <link
@@ -689,5 +685,4 @@
       effort="5"
       velocity="1" />
-    <mimic joint="ServoGear" multiplier="-1"/>
   </joint>
   <gazebo reference="base_link">
