Commit message: All controller have the mimic joints declered but it still doesn't work

File: src/robot_moveit_config/config/armr5.ros2_control.xacro (robot description, xacro)
@@ -50,4 +50,39 @@
                 <state_interface name="velocity"/>
             </joint>
+            <joint name="LeftGripper">
+                <command_interface name="position"/>
+                <state_interface name="position">
+                  <param name="initial_value">${initial_positions['LeftGripper']}</param>
+                </state_interface>
+                <state_interface name="velocity"/>
+            </joint>
+            <joint name="LeftPivotArm">
+                <command_interface name="position"/>
+                <state_interface name="position">
+                  <param name="initial_value">${initial_positions['LeftPivotArm']}</param>
+                </state_interface>
+                <state_interface name="velocity"/>
+            </joint>
+            <joint name="PassifGear">
+                <command_interface name="position"/>
+                <state_interface name="position">
+                  <param name="initial_value">${initial_positions['PassifGear']}</param>
+                </state_interface>
+                <state_ interface name="velocity"/>
+            </joint>
+            <joint name="RightGripper">
+                <command_interface name="position"/>
+                <state_interface name="position">
+                  <param name="initial_value">${initial_positions['RightGripper']}</param>
+                </state_interface>
+                <state_interface name="velocity"/>
+            </joint>
+            <joint name="RightPivotArm">
+                <command_interface name="position"/>
+                <state_interface name="position">
+                  <param name="initial_value">${initial_positions['RightPivotArm']}</param>
+                </state_interface>
+                <state_interface name="velocity"/>
+            </joint>
         </ros2_control>
     </xacro:macro>
